File: PCB/kscan.sch (KiCad schematic (older format))
At the start: 28 parts, among them IC1 ATMEGA328P-A, P1 USB_A, P2 LASER_1, P3 LASER_2, P4 LASER_3, P5 LASER_4, P6 MOTOR_CONN, SW1 RESET, U1 FT232RL, U2 ULN2003A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

Commit message: Adding netlist
Parts:
- C1, C10, C2, C3, C4, C5, C6, C7, C8, C9: footprint (none) -> Capacitors_SMD:C_0805
- D1, D2: footprint (none) -> LEDs:LED_0805
- IC1: footprint TQFP32 -> Housings_QFP:LQFP-32_7x7mm_Pitch0.8mm
- P1: footprint (none) -> Connect:USB_A
- P2, P3, P4, P5: footprint (none) -> Connectors_JST:JST_XH_B02B-XH-A_02x2.50mm_Straight
- P6: footprint (none) -> Connectors_JST:JST_XH_B05B-XH-A_05x2.50mm_Straight
- R1, R2, R3, R4, R5: footprint (none) -> Resistors_SMD:R_0805
- SW1: footprint (none) -> Buttons_Switches_SMD:SW_SPST_B3S-1000
- U1: footprint (none) -> Housings_SSOP:SSOP-28_5.3x10.2mm_Pitch0.65mm
- U2: footprint (none) -> Housings_SOIC:SOIC-16_3.9x9.9mm_Pitch1.27mm
- Y1: footprint (none) -> Crystals:Crystal_SMD_HC49-SD
Other:
- moved on the sheet: C1, C10, C4, C6, C7, D1, D2, P1, P2, P3, P4, P5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

Commit message: Change pin mapping
Parts:
- removed C2: 0.1uF, Capacitors_SMD:C_0805, symbol C_Small
- removed C3: 4.7uF, Capacitors_SMD:C_0805, symbol CP_Small
- D1, D2: symbol LED -> LED-RESCUE-kscan
- P1: symbol USB_A -> USB_A-RESCUE-kscan
Connections:
- net MC1: now reaches U2.1 (I1)
- net MC1: now also IC1.28 ((PCINT13/SCL/ADC5)PC5); no longer IC1.25 ((PCINT10/ADC2)PC2)
- net MC2: now reaches U2.2 (I2)
- net MC2: now also IC1.27 ((PCINT12/SDA/ADC4)PC4); no longer IC1.26 ((PCINT11/ADC3)PC3)
- net MC3: now reaches U2.3 (I3)
- net MC3: now also IC1.26 ((PCINT11/ADC3)PC3); no longer IC1.27 ((PCINT12/SDA/ADC4)PC4)
- net MC4: now reaches U2.4 (I4)
- net MC4: now also IC1.25 ((PCINT10/ADC2)PC2); no longer IC1.28 ((PCINT13/SCL/ADC5)PC5)
